File: UCLED.sch (EAGLE design)
At the start: 36 parts, among them CON1 CON-4P-TABS-JST_GH-RA, CON2 CON-4P-TABS-JST_GH-RA, CON3 PINHEAD_1X06-2, IC1 TJA1051, IC2 STM32F042F4PX, IC3 AP2127-3.3, J1 CONNECTION, J2 CONNECTION

Commit message: updates
Parts:
- removed R1: 1K, R_digikey:1K-5%-0603
Connections:
- removed net N$7: IC2.PB8-BOOT0, R1.2
- net GND: now also IC2.PB8-BOOT0; no longer R1.1
- net USART2_RX: now also CON3.4; no longer CON3.3
- net USART2_TX: now also CON3.3; no longer CON3.4
Changed lines of the file:
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@@
 <part name="GND16" library="supply_symbols" library_urn="urn:adsk.eagle:library:5017758" deviceset="GND" device="" value="GND"/>
 <part name="+P15" library="supply_symbols" library_urn="urn:adsk.eagle:library:5017758" deviceset="3.3V" device=""/>
-<part name="R1" library="R_digikey" library_urn="urn:adsk.eagle:library:2539499" deviceset="1K" device="-0603" package3d_urn="urn:adsk.eagle:package:2539515/2" technology="-5%" value="1K"/>
 <part name="GND17" library="supply_symbols" library_urn="urn:adsk.eagle:library:5017758" deviceset="GND" device="" value="GND"/>
 <part name="+P16" library="supply_symbols" library_urn="urn:adsk.eagle:library:5017758" deviceset="5V" device=""/>
@@
 <attribute name="VALUE" x="152.4" y="143.256" size="1.27" layer="96" font="vector" ratio="15" rot="MR0" align="center"/>
 </instance>
-<instance part="R1" gate="G$1" x="162.56" y="147.32" smashed="yes">
-<attribute name="NAME" x="162.56" y="147.32" size="1.27" layer="95" align="center"/>
-<attribute name="VALUE" x="162.306" y="145.288" size="0.762" layer="96" align="bottom-right"/>
-<attribute name="PACKAGE" x="158.75" y="147.828" size="0.508" layer="95" align="center"/>
-<attribute name="TOLERANCE" x="162.814" y="145.288" size="0.762" layer="96"/>
-</instance>
 <instance part="GND17" gate="1" x="149.86" y="147.32" smashed="yes" rot="R270">
 <attribute name="VALUE" x="148.59" y="147.32" size="1.27" layer="96" font="vector" ratio="15" rot="R270" align="center"/>
@@
 </segment>
 <segment>
-<pinref part="R1" gate="G$1" pin="1"/>
 <pinref part="GND17" gate="1" pin="GND"/>
 <wire x1="152.4" y1="147.32" x2="157.48" y2="147.32" width="0.1524" layer="91"/>
+<pinref part="IC2" gate="G$1" pin="PB8-BOOT0"/>
+<wire x1="170.18" y1="147.32" x2="167.64" y2="147.32" width="0.1524" layer="91"/>
+<wire x1="167.64" y1="147.32" x2="157.48" y2="147.32" width="0.1524" layer="91"/>
 </segment>
 <segment>
@@
 </segment>
 </net>
-<net name="N$7" class="0">
-<segment>
-<pinref part="IC2" gate="G$1" pin="PB8-BOOT0"/>
-<pinref part="R1" gate="G$1" pin="2"/>
-<wire x1="170.18" y1="147.32" x2="167.64" y2="147.32" width="0.1524" layer="91"/>
-</segment>
-</net>
 <net name="SWCLK" class="0">
 <segment>
@@
 </segment>
 <segment>
+<wire x1="238.76" y1="154.94" x2="241.3" y2="154.94" width="0.1524" layer="91"/>
+<label x="238.76" y="154.94" size="1.27" layer="95" font="vector" ratio="15" rot="R180" xref="yes"/>
+<pinref part="CON3" gate="G$1" pin="3"/>
+</segment>
+</net>
+<net name="USART2_RX" class="0">
+<segment>
+<pinref part="IC2" gate="G$1" pin="PA3"/>
+<wire x1="170.18" y1="127" x2="167.64" y2="127" width="0.1524" layer="91"/>
+<label x="167.64" y="127" size="1.27" layer="95" font="vector" ratio="15" rot="R180" xref="yes"/>
+</segment>
+<segment>
 <wire x1="241.3" y1="157.48" x2="238.76" y2="157.48" width="0.1524" layer="91"/>
 <label x="238.76" y="157.48" size="1.27" layer="95" font="vector" ratio="15" rot="R180" xref="yes"/>
@@
 </segment>
 </net>
-<net name="USART2_RX" class="0">
-<segment>
-<pinref part="IC2" gate="G$1" pin="PA3"/>
-<wire x1="170.18" y1="127" x2="167.64" y2="127" width="0.1524" layer="91"/>
-<label x="167.64" y="127" size="1.27" layer="95" font="vector" ratio="15" rot="R180" xref="yes"/>
-</segment>
-<segment>
-<wire x1="238.76" y1="154.94" x2="241.3" y2="154.94" width="0.1524" layer="91"/>
-<label x="238.76" y="154.94" size="1.27" layer="95" font="vector" ratio="15" rot="R180" xref="yes"/>
-<pinref part="CON3" gate="G$1" pin="3"/>
-</segment>
-</net>

Commit message: V0.1 completed
Parts:
- removed CON3: PINHEAD_1X06-2, pinhead:PINHEAD_1X06-2
- added PAD1, PAD2, PAD3, PAD4, PAD5, PAD6: PAD-S_2X2, PADS:PAD-S_2X2
Connections:
- net GND: now also PAD2.P$1; no longer CON3.5
- net SWCLK: now also PAD6.P$1; no longer CON3.1
- net SWDIO: now also PAD5.P$1; no longer CON3.2
- net USART2_RX: now also PAD3.P$1; no longer CON3.4
- net USART2_TX: now also PAD4.P$1; no longer CON3.3
- net VDD_5V: now also PAD1.P$1; no longer CON3.6
Changed lines of the file:
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@@
 <?xml version="1.0" encoding="utf-8"?>
 <!DOCTYPE eagle SYSTEM "eagle.dtd">
-<eagle version="9.3.1">
+<eagle version="9.3.2">
 <drawing>
 <settings>
@@
 <part name="GND17" library="supply_symbols" library_urn="urn:adsk.eagle:library:5017758" deviceset="GND" device="" value="GND"/>
 <part name="+P16" library="supply_symbols" library_urn="urn:adsk.eagle:library:5017758" deviceset="5V" device=""/>
-<part name="CON3" library="pinhead" library_urn="urn:adsk.eagle:library:2540341" deviceset="PINHEAD_1X06" device="-2" package3d_urn="urn:adsk.eagle:package:6650269/2"/>
 <part name="GND18" library="supply_symbols" library_urn="urn:adsk.eagle:library:5017758" deviceset="GND" device="" value="GND"/>
 <part name="C16" library="C_digikey" library_urn="urn:adsk.eagle:library:2539367" deviceset="8PF" device="-0603" package3d_urn="urn:adsk.eagle:package:2539381/2" technology="-25V_10%_X7R" value="8pF"/>
@@
 <part name="CON1" library="Connectors" library_urn="urn:adsk.eagle:library:3750510" deviceset="CON-4P-TABS" device="-RA" package3d_urn="urn:adsk.eagle:package:1040150/6" technology="-JST_GH"/>
 <part name="CON2" library="Connectors" library_urn="urn:adsk.eagle:library:3750510" deviceset="CON-4P-TABS" device="-RA" package3d_urn="urn:adsk.eagle:package:1040150/6" technology="-JST_GH"/>
+<part name="PAD1" library="PADS" library_urn="urn:adsk.eagle:library:3188696" deviceset="PAD" device="-S_2X2" package3d_urn="urn:adsk.eagle:package:3188704/1"/>
+<part name="PAD2" library="PADS" library_urn="urn:adsk.eagle:library:3188696" deviceset="PAD" device="-S_2X2" package3d_urn="urn:adsk.eagle:package:3188704/1"/>
+<part name="PAD3" library="PADS" library_urn="urn:adsk.eagle:library:3188696" deviceset="PAD" device="-S_2X2" package3d_urn="urn:adsk.eagle:package:3188704/1"/>
+<part name="PAD4" library="PADS" library_urn="urn:adsk.eagle:library:3188696" deviceset="PAD" device="-S_2X2" package3d_urn="urn:adsk.eagle:package:3188704/1"/>
+<part name="PAD5" library="PADS" library_urn="urn:adsk.eagle:library:3188696" deviceset="PAD" device="-S_2X2" package3d_urn="urn:adsk.eagle:package:3188704/1"/>
+<part name="PAD6" library="PADS" library_urn="urn:adsk.eagle:library:3188696" deviceset="PAD" device="-S_2X2" package3d_urn="urn:adsk.eagle:package:3188704/1"/>
 </parts>
 <sheets>
@@
 <attribute name="VALUE" x="152.4" y="123.19" size="1.27" layer="96" font="vector" ratio="15" align="center"/>
 </instance>
-<instance part="+P15" gate="G$1" x="152.4" y="139.7" smashed="yes" rot="MR0">
-<attribute name="VALUE" x="152.4" y="143.256" size="1.27" layer="96" font="vector" ratio="15" rot="MR0" align="center"/>
+<instance part="+P15" gate="G$1" x="149.86" y="137.16" smashed="yes" rot="MR270">
+<attribute name="VALUE" x="146.304" y="137.16" size="1.27" layer="96" font="vector" ratio="15" rot="MR270" align="center"/>
 </instance>
 <instance part="GND17" gate="1" x="149.86" y="147.32" smashed="yes" rot="R270">
@@
 <instance part="+P16" gate="G$1" x="233.68" y="165.1" smashed="yes" rot="MR0">
 <attribute name="VALUE" x="233.68" y="168.656" size="1.27" layer="96" font="vector" ratio="15" rot="MR0" align="center"/>
-</instance>
-<instance part="CON3" gate="G$1" x="248.92" y="147.32" smashed="yes" rot="MR0">
-<attribute name="NAME" x="246.38" y="166.37" size="1.778" layer="95" font="vector" ratio="15" rot="MR0" align="center"/>
 </instance>
 <instance part="GND18" gate="1" x="226.06" y="160.02" smashed="yes" rot="R270">
@@
 <instance part="CON2" gate="G$1" x="15.24" y="144.78" smashed="yes" rot="MR270">
 <attribute name="NAME" x="8.89" y="138.43" size="1.778" layer="95" font="vector" ratio="15" rot="MR90" align="center"/>
+</instance>
+<instance part="PAD1" gate="G$1" x="243.84" y="162.56" smashed="yes" rot="MR0">
+<attribute name="NAME" x="243.84" y="163.83" size="1.27" layer="95" font="vector" ratio="15" rot="MR0" align="center"/>
+</instance>
+<instance part="PAD2" gate="G$1" x="243.84" y="160.02" smashed="yes" rot="MR0">
+<attribute name="NAME" x="243.84" y="161.29" size="1.27" layer="95" font="vector" ratio="15" rot="MR0" align="center"/>
+</instance>
+<instance part="PAD3" gate="G$1" x="243.84" y="157.48" smashed="yes" rot="MR0">
+<attribute name="NAME" x="243.84" y="158.75" size="1.27" layer="95" font="vector" ratio="15" rot="MR0" align="center"/>
+</instance>
+<instance part="PAD4" gate="G$1" x="243.84" y="154.94" smashed="yes" rot="MR0">
+<attribute name="NAME" x="243.84" y="156.21" size="1.27" layer="95" font="vector" ratio="15" rot="MR0" align="center"/>
+</instance>
+<instance part="PAD5" gate="G$1" x="243.84" y="152.4" smashed="yes" rot="MR0">
+<attribute name="NAME" x="243.84" y="153.67" size="1.27" layer="95" font="vector" ratio="15" rot="MR0" align="center"/>
+</instance>
+<instance part="PAD6" gate="G$1" x="243.84" y="149.86" smashed="yes" rot="MR0">
+<attribute name="NAME" x="243.84" y="151.13" size="1.27" layer="95" font="vector" ratio="15" rot="MR0" align="center"/>
 </instance>
 </instances>
@@
 </segment>
 <segment>
-<pinref part="CON3" gate="G$1" pin="5"/>
 <pinref part="GND18" gate="1" pin="GND"/>
 <wire x1="241.3" y1="160.02" x2="228.6" y2="160.02" width="0.1524" layer="91"/>
+<pinref part="PAD2" gate="G$1" pin="P$1"/>
 </segment>
 <segment>
@@
 <pinref part="+P16" gate="G$1" pin="VDD_5V"/>
 <wire x1="233.68" y1="162.56" x2="233.68" y2="165.1" width="0.1524" layer="91"/>
-<pinref part="CON3" gate="G$1" pin="6"/>
 <wire x1="236.22" y1="162.56" x2="241.3" y2="162.56" width="0.1524" layer="91"/>
+<pinref part="PAD1" gate="G$1" pin="P$1"/>
 </segment>
 </net>
@@
 <pinref part="C15" gate="G$1" pin="2"/>
 <wire x1="152.4" y1="134.62" x2="152.4" y2="137.16" width="0.1524" layer="91"/>
-<wire x1="152.4" y1="137.16" x2="152.4" y2="139.7" width="0.1524" layer="91"/>
+<wire x1="152.4" y1="137.16" x2="149.86" y2="137.16" width="0.1524" layer="91"/>
 <junction x="152.4" y="137.16"/>
 <pinref part="+P15" gate="G$1" pin="VDD_3V3"/>
@@
 <wire x1="241.3" y1="149.86" x2="238.76" y2="149.86" width="0.1524" layer="91"/>
 <label x="238.76" y="149.86" size="1.27" layer="95" font="vector" ratio="15" rot="R180" xref="yes"/>
-<pinref part="CON3" gate="G$1" pin="1"/>
+<pinref part="PAD6" gate="G$1" pin="P$1"/>
 </segment>
 </net>
@@
 <wire x1="241.3" y1="152.4" x2="238.76" y2="152.4" width="0.1524" layer="91"/>
 <label x="238.76" y="152.4" size="1.27" layer="95" font="vector" ratio="15" rot="R180" xref="yes"/>
-<pinref part="CON3" gate="G$1" pin="2"/>
+<pinref part="PAD5" gate="G$1" pin="P$1"/>
 </segment>
 </net>
@@
 <wire x1="238.76" y1="154.94" x2="241.3" y2="154.94" width="0.1524" layer="91"/>
 <label x="238.76" y="154.94" size="1.27" layer="95" font="vector" ratio="15" rot="R180" xref="yes"/>
-<pinref part="CON3" gate="G$1" pin="3"/>
+<pinref part="PAD4" gate="G$1" pin="P$1"/>
 </segment>
 </net>
@@
 <wire x1="241.3" y1="157.48" x2="238.76" y2="157.48" width="0.1524" layer="91"/>
 <label x="238.76" y="157.48" size="1.27" layer="95" font="vector" ratio="15" rot="R180" xref="yes"/>
-<pinref part="CON3" gate="G$1" pin="4"/>
+<pinref part="PAD3" gate="G$1" pin="P$1"/>
 </segment>
 </net>
@@
 <pinref part="Z1" gate="P" pin="2"/>
 <wire x1="132.08" y1="146.05" x2="132.08" y2="149.86" width="0.1524" layer="91"/>
-<wire x1="132.08" y1="149.86" x2="142.24" y2="149.86" width="0.1524" layer="91"/>
+<wire x1="132.08" y1="149.86" x2="144.78" y2="149.86" width="0.1524" layer="91"/>
 <pinref part="C17" gate="G$1" pin="2"/>
 <wire x1="132.08" y1="149.86" x2="129.54" y2="149.86" width="0.1524" layer="91"/>
 <junction x="132.08" y="149.86"/>
 <pinref part="IC2" gate="G$1" pin="PF0"/>
-<wire x1="170.18" y1="144.78" x2="147.32" y2="144.78" width="0.1524" layer="91"/>
-<wire x1="147.32" y1="144.78" x2="147.32" y2="149.86" width="0.1524" layer="91"/>
-<wire x1="147.32" y1="149.86" x2="142.24" y2="149.86" width="0.1524" layer="91"/>
+<wire x1="170.18" y1="144.78" x2="144.78" y2="144.78" width="0.1524" layer="91"/>
+<wire x1="144.78" y1="144.78" x2="144.78" y2="149.86" width="0.1524" layer="91"/>
 </segment>
 </net>
@@
 <junction x="132.08" y="137.16"/>
 <pinref part="IC2" gate="G$1" pin="PF1"/>
-<wire x1="170.18" y1="142.24" x2="147.32" y2="142.24" width="0.1524" layer="91"/>
-<wire x1="147.32" y1="142.24" x2="147.32" y2="137.16" width="0.1524" layer="91"/>
-<wire x1="147.32" y1="137.16" x2="144.78" y2="137.16" width="0.1524" layer="91"/>
+<wire x1="170.18" y1="142.24" x2="144.78" y2="142.24" width="0.1524" layer="91"/>
+<wire x1="144.78" y1="142.24" x2="144.78" y2="137.16" width="0.1524" layer="91"/>
 </segment>
 </net>
@@
 </sheet>
 </sheets>
+<errors>
+</errors>
 </schematic>
 </drawing>

Commit message: attribute fixes
Parts:
- added FD1, FD2: FIDUCIALMOUNT, misc:FIDUCIALMOUNT
- IC2: DIGIKEY# (none) -> 497-17343-ND
Changed lines of the file:
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@@
 </attributes>
 <variantdefs>
+<variantdef name="BASIC" current="yes"/>
 </variantdefs>
 <classes>
@@
 <part name="GND3" library="supply_symbols" library_urn="urn:adsk.eagle:library:5017758" deviceset="GND" device="" value="GND"/>
 <part name="+P1" library="supply_symbols" library_urn="urn:adsk.eagle:library:5017758" deviceset="5V" device=""/>
-<part name="IC2" library="stm32" library_urn="urn:adsk.eagle:library:2473361" deviceset="STM32F042F4PX" device="" package3d_urn="urn:adsk.eagle:package:2473346/4"/>
+<part name="IC2" library="stm32" library_urn="urn:adsk.eagle:library:2473361" deviceset="STM32F042F4PX" device="" package3d_urn="urn:adsk.eagle:package:2473346/4">
+<attribute name="DIGIKEY#" value="497-17343-ND"/>
+</part>
 <part name="LED1" library="misc" library_urn="urn:adsk.eagle:library:5347860" deviceset="WS2812B" device="" package3d_urn="urn:adsk.eagle:package:8849294/2"/>
 <part name="+P2" library="supply_symbols" library_urn="urn:adsk.eagle:library:5017758" deviceset="5V" device=""/>
@@
 <part name="Z1" library="myxa_masterlib" library_urn="urn:adsk.eagle:library:1040030" deviceset="CRYSTAL" device="-NX3225GD" package3d_urn="urn:adsk.eagle:package:1040148/2" value="8MHz"/>
 <part name="GND19" library="supply_symbols" library_urn="urn:adsk.eagle:library:5017758" deviceset="GND" device="" value="GND"/>
-<part name="J1" library="misc" library_urn="urn:adsk.eagle:library:5347860" deviceset="CONNECTION" device="" package3d_urn="urn:adsk.eagle:package:7439847/1"/>
+<part name="J1" library="misc" library_urn="urn:adsk.eagle:library:5347860" deviceset="CONNECTION" device="" package3d_urn="urn:adsk.eagle:package:7439847/1">
+<variant name="BASIC" populate="no"/>
+</part>
 <part name="GND20" library="supply_symbols" library_urn="urn:adsk.eagle:library:5017758" deviceset="GND" device="" value="GND"/>
-<part name="J2" library="misc" library_urn="urn:adsk.eagle:library:5347860" deviceset="CONNECTION" device="" package3d_urn="urn:adsk.eagle:package:7439847/1"/>
+<part name="J2" library="misc" library_urn="urn:adsk.eagle:library:5347860" deviceset="CONNECTION" device="" package3d_urn="urn:adsk.eagle:package:7439847/1">
+<variant name="BASIC" populate="no"/>
+</part>
 <part name="GND22" library="supply_symbols" library_urn="urn:adsk.eagle:library:5017758" deviceset="GND" device="" value="GND"/>
 <part name="GND23" library="supply_symbols" library_urn="urn:adsk.eagle:library:5017758" deviceset="GND" device="" value="GND"/>
 <part name="CON1" library="Connectors" library_urn="urn:adsk.eagle:library:3750510" deviceset="CON-4P-TABS" device="-RA" package3d_urn="urn:adsk.eagle:package:1040150/6" technology="-JST_GH"/>
 <part name="CON2" library="Connectors" library_urn="urn:adsk.eagle:library:3750510" deviceset="CON-4P-TABS" device="-RA" package3d_urn="urn:adsk.eagle:package:1040150/6" technology="-JST_GH"/>
-<part name="PAD1" library="PADS" library_urn="urn:adsk.eagle:library:3188696" deviceset="PAD" device="-S_2X2" package3d_urn="urn:adsk.eagle:package:3188704/1"/>
-<part name="PAD2" library="PADS" library_urn="urn:adsk.eagle:library:3188696" deviceset="PAD" device="-S_2X2" package3d_urn="urn:adsk.eagle:package:3188704/1"/>
-<part name="PAD3" library="PADS" library_urn="urn:adsk.eagle:library:3188696" deviceset="PAD" device="-S_2X2" package3d_urn="urn:adsk.eagle:package:3188704/1"/>
-<part name="PAD4" library="PADS" library_urn="urn:adsk.eagle:library:3188696" deviceset="PAD" device="-S_2X2" package3d_urn="urn:adsk.eagle:package:3188704/1"/>
-<part name="PAD5" library="PADS" library_urn="urn:adsk.eagle:library:3188696" deviceset="PAD" device="-S_2X2" package3d_urn="urn:adsk.eagle:package:3188704/1"/>
-<part name="PAD6" library="PADS" library_urn="urn:adsk.eagle:library:3188696" deviceset="PAD" device="-S_2X2" package3d_urn="urn:adsk.eagle:package:3188704/1"/>
+<part name="PAD1" library="PADS" library_urn="urn:adsk.eagle:library:3188696" deviceset="PAD" device="-S_2X2" package3d_urn="urn:adsk.eagle:package:3188704/1">
+<variant name="BASIC" populate="no"/>
+</part>
+<part name="PAD2" library="PADS" library_urn="urn:adsk.eagle:library:3188696" deviceset="PAD" device="-S_2X2" package3d_urn="urn:adsk.eagle:package:3188704/1">
+<variant name="BASIC" populate="no"/>
+</part>
+<part name="PAD3" library="PADS" library_urn="urn:adsk.eagle:library:3188696" deviceset="PAD" device="-S_2X2" package3d_urn="urn:adsk.eagle:package:3188704/1">
+<variant name="BASIC" populate="no"/>
+</part>
+<part name="PAD4" library="PADS" library_urn="urn:adsk.eagle:library:3188696" deviceset="PAD" device="-S_2X2" package3d_urn="urn:adsk.eagle:package:3188704/1">
+<variant name="BASIC" populate="no"/>
+</part>
+<part name="PAD5" library="PADS" library_urn="urn:adsk.eagle:library:3188696" deviceset="PAD" device="-S_2X2" package3d_urn="urn:adsk.eagle:package:3188704/1">
+<variant name="BASIC" populate="no"/>
+</part>
+<part name="PAD6" library="PADS" library_urn="urn:adsk.eagle:library:3188696" deviceset="PAD" device="-S_2X2" package3d_urn="urn:adsk.eagle:package:3188704/1">
+<variant name="BASIC" populate="no"/>
+</part>
+<part name="FD1" library="misc" library_urn="urn:adsk.eagle:library:5347860" deviceset="FIDUCIALMOUNT" device="" package3d_urn="urn:adsk.eagle:package:7544833/1">
+<variant name="BASIC" populate="no"/>
+</part>
+<part name="FD2" library="misc" library_urn="urn:adsk.eagle:library:5347860" deviceset="FIDUCIALMOUNT" device="" package3d_urn="urn:adsk.eagle:package:7544833/1">
+<variant name="BASIC" populate="no"/>
+</part>
 </parts>
 <sheets>
@@
 <attribute name="NAME" x="243.84" y="151.13" size="1.27" layer="95" font="vector" ratio="15" rot="MR0" align="center"/>
 </instance>
+<instance part="FD1" gate="G$1" x="12.7" y="106.68" smashed="yes"/>
+<instance part="FD2" gate="G$1" x="12.7" y="99.06" smashed="yes"/>
 </instances>
 <busses>
